File: hardware/Autonomous_Sailboat/Autonomous_Sailboat.kicad_sch (KiCad schematic)
At the start: 16 parts, among them Q1 Q_NMOS, U1 STM32H755ZITx

Commit message: preliminary implementation of the battery sensor
Parts:
- removed PullDown: 10k, symbol Device:R
- removed Q1: Q_NMOS, symbol Device:Q_NMOS
- removed R_Gate: 220, symbol Device:R
Connections:
- net GND: now also R_B1-.2, R_B2-.2, R_B3-.2, R_B4-.2
- no-connect marks 103 -> 104

Commit message: moved the telemetry all into a shared file
Connections:
- net sensorEncoder_I2C1SCL: now reaches U1.133 (PB6)
- net sensorEncoder_I2C1SDA: now reaches U1.134 (PB7)
- net B1_UserButton: no longer names the net of U1.9 (PC13)
- net GPIO_SailServoControl: no longer names the net of U1.59 (PE9)
- net I2C2_SCL: no longer names the net of U1.66 (PB10)
- net I2C2_SDA: no longer names the net of U1.67 (PB11)
- net LD1_liveliness renamed live_LEDGreen
- net LD3_UserButtonLED: no longer names the net of U1.74 (PB14)
- net UART4RX_WindSensor: no longer names the net of U1.110 (PC11)
- net UART4TX_WindSensort: no longer names the net of U1.109 (PC10)
- net UART7RX_GPS: no longer names the net of U1.20 (PF6)
- net UART7TX_GPS: no longer names the net of U1.21 (PF7)
- no-connect marks 104 -> 102
Changed lines of the file:
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@@
-	)
-	(no_connect
-		(at 323.85 167.64)
 	)
 	(no_connect
@@
 	)
 	(no_connect
-		(at 323.85 170.18)
-	)
-	(no_connect
 		(at 237.49 121.92)
 	)
@@
 	(wire
 		(pts
+			(xy 323.85 167.64) (xy 330.2 167.64)
+		)
+		(stroke
+			(width 0)
+			(type default)
+		)
+	)
+	(wire
+		(pts
 			(xy 369.57 124.46) (xy 419.1 124.46)
 		)
@@
 	(wire
 		(pts
-			(xy 323.85 180.34) (xy 342.9 180.34)
+			(xy 330.2 167.64) (xy 330.2 165.1)
 		)
 		(stroke
@@
 	(wire
 		(pts
-			(xy 215.9 213.36) (xy 237.49 213.36)
-		)
-		(stroke
-			(width 0)
-			(type default)
-		)
-	)
-	(wire
-		(pts
-			(xy 215.9 172.72) (xy 228.6 172.72)
-		)
-		(stroke
-			(width 0)
-			(type default)
-		)
-	)
-	(wire
-		(pts
-			(xy 323.85 228.6) (xy 342.9 228.6)
-		)
-		(stroke
-			(width 0)
-			(type default)
-		)
-	)
-	(wire
-		(pts
 			(xy 323.85 109.22) (xy 331.47 109.22)
 		)
@@
 	(wire
 		(pts
-			(xy 323.85 223.52) (xy 342.9 223.52)
-		)
-		(stroke
-			(width 0)
-			(type default)
-		)
-	)
-	(wire
-		(pts
 			(xy 381 109.22) (xy 381 129.54)
 		)
@@
 	(wire
 		(pts
-			(xy 330.2 218.44) (xy 342.9 218.44)
-		)
-		(stroke
-			(width 0)
-			(type default)
-		)
-	)
-	(wire
-		(pts
 			(xy 419.1 124.46) (xy 419.1 129.54)
 		)
@@
 	(wire
 		(pts
+			(xy 323.85 170.18) (xy 342.9 170.18)
+		)
+		(stroke
+			(width 0)
+			(type default)
+		)
+	)
+	(wire
+		(pts
 			(xy 323.85 121.92) (xy 356.87 121.92)
 		)
@@
 	(wire
 		(pts
-			(xy 323.85 187.96) (xy 342.9 187.96)
-		)
-		(stroke
-			(width 0)
-			(type default)
-		)
-	)
-	(wire
-		(pts
 			(xy 393.7 137.16) (xy 400.05 137.16)
 		)
@@
 	(wire
 		(pts
-			(xy 323.85 220.98) (xy 330.2 220.98)
-		)
-		(stroke
-			(width 0)
-			(type default)
-		)
-	)
-	(wire
-		(pts
 			(xy 283.21 99.06) (xy 285.75 99.06)
 		)
@@
 	(wire
 		(pts
-			(xy 330.2 177.8) (xy 330.2 175.26)
-		)
-		(stroke
-			(width 0)
-			(type default)
-		)
-	)
-	(wire
-		(pts
 			(xy 323.85 119.38) (xy 344.17 119.38)
 		)
@@
 	(wire
 		(pts
-			(xy 323.85 177.8) (xy 330.2 177.8)
-		)
-		(stroke
-			(width 0)
-			(type default)
-		)
-	)
-	(wire
-		(pts
 			(xy 419.1 104.14) (xy 419.1 124.46)
 		)
@@
 	(wire
 		(pts
-			(xy 228.6 170.18) (xy 228.6 172.72)
-		)
-		(stroke
-			(width 0)
-			(type default)
-		)
-	)
-	(wire
-		(pts
 			(xy 393.7 104.14) (xy 393.7 119.38)
 		)
@@
 	(wire
 		(pts
-			(xy 215.9 167.64) (xy 237.49 167.64)
+			(xy 330.2 165.1) (xy 342.9 165.1)
 		)
 		(stroke
@@
 	(wire
 		(pts
-			(xy 330.2 175.26) (xy 342.9 175.26)
-		)
-		(stroke
-			(width 0)
-			(type default)
-		)
-	)
-	(wire
-		(pts
 			(xy 50.8 50.8) (xy 558.8 50.8)
 		)
@@
 		(pts
 			(xy 273.05 99.06) (xy 275.59 99.06)
-		)
-		(stroke
-			(width 0)
-			(type default)
-		)
-	)
-	(wire
-		(pts
-			(xy 330.2 220.98) (xy 330.2 218.44)
-		)
-		(stroke
-			(width 0)
-			(type default)
-		)
-	)
-	(wire
-		(pts
-			(xy 237.49 170.18) (xy 228.6 170.18)
 		)
 		(stroke
@@
 		)
 	)
-	(label "LD1_liveliness"
+	(label "live_LEDGreen"
 		(at 342.9 152.4 0)
-		(effects
-			(font
-				(size 1.27 1.27)
-			)
-			(justify left bottom)
-		)
-	)
-	(label "UART7RX_GPS"
-		(at 215.9 167.64 0)
-		(effects
-			(font
-				(size 1.27 1.27)
-			)
-			(justify left bottom)
-		)
-	)
-	(label "UART4RX_WindSensor"
-		(at 342.9 223.52 0)
 		(effects
 			(font
@@
 		)
 	)
-	(label "I2C2_SDA"
-		(at 342.9 180.34 0)
-		(effects
-			(font
-				(size 1.27 1.27)
-			)
-			(justify left bottom)
-		)
-	)
-	(label "UART7TX_GPS"
-		(at 215.9 172.72 0)
-		(effects
-			(font
-				(size 1.27 1.27)
-			)
-			(justify left bottom)
-		)
-	)
-	(label "LD3_UserButtonLED"
-		(at 342.9 187.96 0)
-		(effects
-			(font
-				(size 1.27 1.27)
-			)
-			(justify left bottom)
-		)
-	)
-	(label "UART4TX_WindSensort"
-		(at 342.9 218.44 0)
-		(effects
-			(font
-				(size 1.27 1.27)
-			)
-			(justify left bottom)
-		)
-	)
-	(label "B1_UserButton"
-		(at 342.9 228.6 0)
+	(label "sensorEncoder_I2C1SCL"
+		(at 342.9 165.1 0)
 		(effects
 			(font
@@
 		)
 	)
+	(label "sensorEncoder_I2C1SDA"
+		(at 342.9 170.18 0)
+		(effects
+			(font
+				(size 1.27 1.27)
+			)
+			(justify left bottom)
+		)
+	)
 	(label "B0"
 		(at 368.3 96.52 0)
@@
 		)
 	)
-	(label "I2C2_SCL"
-		(at 342.9 175.26 0)
-		(effects
-			(font
-				(size 1.27 1.27)
-			)
-			(justify left bottom)
-		)
-	)
 	(label "B2"
 		(at 393.7 96.52 0)
@@
 		)
 	)
-	(label "GPIO_SailServoControl"
-		(at 215.9 213.36 180)
-		(effects
-			(font
-				(size 1.27 1.27)
-			)
-			(justify right bottom)
-		)
-	)
