File: hardware/Autonomous_Sailboat/Autonomous_Sailboat.kicad_sch (KiCad schematic)
At the start: 13 parts, among them U1 STM32H755ZITx

Commit message: fixed the stack problem, probably
Connections:
- net at C_filterB3.2, R_B3+.2, R_B3-.1: now also U1.45 (PA6); no longer U1.44 (PA5)
- net at C_filterB1.2, R_B1+.2, R_B1-.1: now also U1.43 (PA4); no longer U1.37 (PA0)
- net at C_filterB2.2, R_B2+.2, R_B2-.1: now also U1.44 (PA5); no longer U1.43 (PA4)
- net at C_filterB4.2, R_B4+.2, R_B4-.1: now also U1.46 (PA7); no longer U1.45 (PA6)
- no-connect marks 100 -> 103
Other:
- moved on the sheet: C_filterB1, C_filterB2, C_filterB3, C_filterB4, R_B1+, R_B1-, R_B2+, R_B2-, R_B3+, R_B3-, R_B4+, R_B4-
